File: hardware/blackpkb/blackpkb.kicad_sch (KiCad schematic)
At the start: 30 parts, among them SW1 SW_Push_45deg, SW10 SW_Push_45deg, SW11 SW_Push_45deg, SW12 SW_Push_45deg, SW13 RotaryEncoder_Switch, SW2 SW_Push_45deg, SW3 SW_Push_45deg, SW4 SW_Push_45deg, SW5 SW_Push_45deg, SW6 SW_Push_45deg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

Commit message: section the schematic. Add infomations, remove redundant files
Other:
- note added: "Keyboard"
- note added: "MCU"
- note added: "Mounting Holes"
- note added: "Rotary Encoder"
- company: (none) -> author - alcato
- title: (none) -> blackpkb
- moved on the sheet: H1, H2, H3, H4, SW1, SW10, SW11, SW12, SW13, SW2, SW3, SW4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

Commit message: hardware v0.2
Parts:
- removed D10, D11, D12, D4, D8, D9: 1N4148, Diode_THT:D_DO-35_SOD27_P7.62mm_Horizontal, symbol Diode:1N4148
- removed SW10, SW11, SW12, SW4, SW8, SW9: SW_Push_45deg, Button_Switch_Keyboard:SW_Cherry_MX_1.00u_PCB, symbol Switch:SW_Push_45deg
- added D4, D8, D9: LED_Small, LED_THT:LED_D3.0mm, symbol Device:LED_Small
- added R1, R2, R3: 330, Resistor_THT:R_Axial_DIN0207_L6.3mm_D2.5mm_P7.62mm_Horizontal, symbol Device:R_Small
Connections:
- net +3.3V: now reaches U1.20 (3V3)
- net +3.3V: now also R1.1, R2.1, R3.1
- net LED_RED: now reaches U1.26 (PA0)
- net LED_RED: now also D9.1 (K)
- net LED_GREEN: now reaches U1.27 (PA1)
- net LED_GREEN: now also D8.1 (K)
- net LED_YELLOW: now reaches U1.28 (PA2)
- net LED_YELLOW: now also D4.1 (K)
- net COL_4: no longer names the net of U1.4 (PB15)
- net ROW_3: no longer names the net of U1.13 (PB5)
- new net: D4.2 (A), R1.2
- new net: D8.2 (A), R2.2
- new net: D9.2 (A), R3.2
- no-connect marks 32 -> 30
